Commit message: Publish portable Zekeeparm update on 1022

File: src/zekeep_bringup/description/urdf/sixaxis.urdf (robot description, URDF)
Before this commit: robot zk_xm115_00_description, 11 links, 10 joints
Links:
- added link official_tcp
Joints:
- added joint official_tcp_fixed: type fixed, parent link6, child official_tcp, origin xyz=0 0 0.15539 rpy=0 -1.5708 3.1415
- joint gripper_joint: limit lower=0 upper=0.035 effort=10 velocity=0.05 -> lower=0 upper=0.03258620689655173 effort=10 velocity=0.05
- joint joint3: limit lower=0 upper=3.7 effort=27 velocity=8 -> lower=-0.01 upper=3.7 effort=27 velocity=8
- joint right_joint: limit lower=0 upper=0.035 effort=10 velocity=0.05 -> lower=0 upper=0.03258620689655173 effort=10 velocity=0.05
